Commit message: redid package structure

File: linear_slider_description/config/linear_slider.ros2_control.xacro (robot description, xacro)
@@ -9,12 +9,12 @@
             </hardware>
             <joint name="ls_base_link_ls_moving_base_joint">
-                <command_interface name="position"/>
+                <!-- <command_interface name="position"/> -->
                 <command_interface name="velocity"/>
-                <command_interface name="effort"/>
-                <state_interface name="position">
+                <!-- <command_interface name="effort"/> -->
+                <!-- <state_interface name="position">
                   <param name="initial_value">${initial_positions['ls_base_link_ls_moving_base_joint']}</param>
-                </state_interface>
+                </state_interface> -->
                 <state_interface name="velocity"/>
-                <state_interface name="effort"/>
+                <!-- <state_interface name="effort"/> -->
             </joint>
         </ros2_control>

File: linear_slider_description/urdf/linear_slider.urdf (robot description, URDF)
Before this commit: robot linear_slider, 2 links, 1 joints
Links:
- link base_link: geometry visual mesh filename=package://linear-slider/linear_slider_description/meshes/7t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 scale=0.001 0.001 0.001
- link ls_moving_base: geometry collision mesh filename=package://linear-slider/linear_slider_description/meshes/7t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 scale=0.001 0.001 0.001; visual mesh filename=package://linear-slider/linear_slider_description/meshes/7t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 scale=0.001 0.001 0.001

File: linear_slider_description/urdf/linear_slider_urdf.xacro (robot description, xacro)
@@ -37,5 +37,5 @@
             <origin rpy="${base_link_start_orientation}" xyz="${start_offset}"/>
             <geometry>
-                <mesh filename="package://linear-slider/meshes/7thlink_fixed.STL" scale="${model_scale}" />
+                <mesh filename="package://linear-slider/linear_slider_description/meshes/7thlink_fixed.STL" scale="${model_scale}" />
             </geometry>
         </visual>
@@ -46,10 +46,14 @@
             <material name="red_v" />
             <geometry>
-                <mesh filename="package://linear-slider/meshes/7thlink_move.STL" scale="${model_scale}" />
+                <mesh
+                    filename="package://linear-slider/linear_slider_description/meshes/7thlink_move.STL"
+                    scale="${model_scale}" />
             </geometry>
         </visual>
         <collision>
             <geometry>
-                <mesh filename="package://linear-slider/meshes/7thlink_move.STL" scale="${model_scale}" />
+                <mesh
+                    filename="package://linear-slider/linear_slider_description/meshes/7thlink_move.STL"
+                    scale="${model_scale}" />
             </geometry>
         </collision>

Commit message: made some big changes to the xacro files. Following the steps of a tutorial (finallY)

File: linear_slider_description/config/linear_slider.ros2_control.xacro (robot description, xacro)
@@ -13,5 +13,5 @@
                 <!-- <plugin>mock_components/GenericSystem</plugin> -->
             </hardware>
-            <joint name="ls_base_link_ls_moving_base_joint">
+            <joint name="base_platform_prismatic_joint">
                 <!-- <command_interface name="position"/> -->
                 <command_interface name="velocity">

File: linear_slider_description/urdf/linear_slider.urdf (robot description, URDF)
Before this commit: robot linear_slider, 2 links, 1 joints
Links:
- link base_link: geometry collision mesh filename=package://linear_slider_description/meshes/7thlink_fixed.STL scale=0.001 0.001 0.001; visual mesh filename=package://linear_slider_description/meshes/7thlink_fixed.STL scale=0.001 0.001 0.001
Joints:
- removed joint ls_base_link_ls_moving_base_joint
- added joint base_platform_prismatic_joint: type prismatic, parent base_link, child ls_moving_base, origin xyz=0.0 0.0 0.0, axis 1 0 0, limit lower=-0.4 upper=0.4 effort=10 velocity=0.25

File: linear_slider_description/urdf/linear_slider/linear_slider_macro.xacro (robot description, xacro)
@@ -40,4 +40,13 @@
             </geometry>
         </visual>
+        <collision>
+            <geometry>
+                <!-- <box size="0.22 0.202 0.118"/> -->
+                <mesh
+                    filename="package://linear_slider_description/meshes/7thlink_fixed.STL"
+                    scale="${model_scale}"
+                />
+            </geometry>
+        </collision>
     </link>
     <link name="ls_moving_base">
@@ -48,5 +57,6 @@
                 <mesh
                     filename="package://linear_slider_description/meshes/7thlink_move.STL"
-                    scale="${model_scale}" />
+                    scale="${model_scale}"
+                />
             </geometry>
         </visual>
@@ -71,5 +81,5 @@
         </inertial>
     </link>
-        <joint name="ls_base_link_ls_moving_base_joint" type="prismatic">
+        <joint name="base_platform_prismatic_joint" type="prismatic">
             <parent link="base_link"/>
             <child link="ls_moving_base"/>
