Commit message: edited some directories. read/write still not working

File: linear_slider_description/config/linear_slider.urdf.xacro (robot description, xacro)
@@ -3,5 +3,5 @@
     <xacro:arg name="initial_positions_file" default="initial_positions.yaml" />
     <!-- Import linear_slider urdf file -->
-    <xacro:include filename="$(find linear-slider)/urdf/linear_slider.urdf" />
+    <xacro:include filename="$(find linear_slider_description)/urdf/linear_slider.urdf" />
     <!-- Import control_xacro -->
     <xacro:include filename="linear_slider.ros2_control.xacro" />

File: linear_slider_description/urdf/linear_slider.urdf (robot description, URDF)
Before this commit: robot linear_slider, 2 links, 1 joints
Links:
- link base_link: geometry visual mesh filename=package://linear_slider_description/meshes/7thlink_fixed.STL scale=0.001 0.001 0.001
- link ls_moving_base: geometry collision mesh filename=package://linear_slider_description/meshes/7thlink_move.STL scale=0.001 0.001 0.001; visual mesh filename=package://linear_slider_description/meshes/7thlink_move.STL scale=0.001 0.001 0.001

File: linear_slider_description/urdf/linear_slider_urdf.xacro (robot description, xacro)
@@ -37,5 +37,5 @@
             <origin rpy="${base_link_start_orientation}" xyz="${start_offset}"/>
             <geometry>
-                <mesh filename="package://linear-slider/linear_slider_description/meshes/7thlink_fixed.STL" scale="${model_scale}" />
+                <mesh filename="package://linear_slider_description/meshes/7thlink_fixed.STL" scale="${model_scale}" />
             </geometry>
         </visual>
@@ -47,5 +47,5 @@
             <geometry>
                 <mesh
-                    filename="package://linear-slider/linear_slider_description/meshes/7thlink_move.STL"
+                    filename="package://linear_slider_description/meshes/7thlink_move.STL"
                     scale="${model_scale}" />
             </geometry>
@@ -54,5 +54,5 @@
             <geometry>
                 <mesh
-                    filename="package://linear-slider/linear_slider_description/meshes/7thlink_move.STL"
+                    filename="package://linear_slider_description/meshes/7thlink_move.STL"
                     scale="${model_scale}" />
             </geometry>

Commit message: fixed some issues in description package. Added base for bringup package

File: linear_slider_description/config/linear_slider.urdf.xacro (robot description, xacro)
@@ -1,9 +1,9 @@
 <?xml version="1.0"?>
 <robot xmlns:xacro="http://www.ros.org/wiki/xacro" name="linear_slider">
-    <xacro:arg name="initial_positions_file" default="initial_positions.yaml" />
+    <xacro:arg name="initial_state_file" default="initial_state.yaml" />
     <!-- Import linear_slider urdf file -->
     <xacro:include filename="$(find linear_slider_description)/urdf/linear_slider.urdf" />
     <!-- Import control_xacro -->
     <xacro:include filename="linear_slider.ros2_control.xacro" />
-    <xacro:linear_slider_ros2_control name="FakeSystem" initial_positions_file="$(arg initial_positions_file)"/>
+    <xacro:linear_slider_ros2_control name="FakeSystem" initial_state_file="$(arg initial_state_file)"/>
 </robot>

File: linear_slider_description/urdf/linear_slider.urdf.xacro (robot description, xacro)
@@ -8,9 +8,10 @@
     <xacro:include filename="$(find linear_slider_description)/urdf/linear_slider/linear_slider_macro.xacro"/>
     <xacro:include filename="$(find linear_slider_description)/urdf/linear_slider/linear_slider.ros2_control.xacro"/>
+    <create />
     <!-- ros2_control -->
     <xacro:linear_slider_ros2_control
         name="linear_slider"
         prefix="$(arg prefix)"
-        initial_positions_file="$(find linear_slider_description)/config/initial_positions.yaml"
+        initial_state_file="$(find linear_slider_description)/config/initial_state.yaml"
         use_mock_hardware="$(arg use_mock_hardware)"
         mock_sensor_commands="$(arg mock_sensor_commands)"

File: linear_slider_description/urdf/linear_slider/linear_slider.ros2_control.xacro (robot description, xacro)
@@ -1,15 +1,16 @@
 <?xml version="1.0"?>
 <robot xmlns:xacro="http://www.ros.org/wiki/xacro">
-    <xacro:macro name="linear_slider_ros2_control" params="name prefix initial_positions_file use_mock_hardware:=^|false mock_sensor_commands:=^|false">
-        <xacro:property name="initial_positions" value="${xacro.load_yaml(initial_positions_file)['initial_positions']}"/>
+    <xacro:macro name="linear_slider_ros2_control" params="name prefix initial_state_file use_mock_hardware:=^|false mock_sensor_commands:=^|false">
+        <xacro:property name="initial_state" value="${xacro.load_yaml(initial_state_file)['initial_state']}"/>
         <ros2_control name="${name}" type="system">
             <!-- Hardware -->
             <hardware>
+                <!-- By default, set up controllers for simulation. This won't work on real hardware -->
+                <plugin>mock_components/GenericSystem</plugin>
+                <param name="mock_sensor_commands">${mock_sensor_commands}</param>
                 <plugin>linear_slider_system_interface/LinearSliderSystemInterface</plugin>
                 <param name="device_name">linear_slider_ros2_control</param>
                 <param name="joint_name">prismatic_joint</param>
                 <param name="robot_ip">169.254.97.178</param>
-                <!-- By default, set up controllers for simulation. This won't work on real hardware -->
-                <!-- <plugin>mock_components/GenericSystem</plugin> -->
             </hardware>
             <!-- Joints -->
@@ -26,14 +27,20 @@
                 <!-- State interface -->
                 <state_interface name="position">
-                  <param name="initial_value">${initial_positions['base_platform_prismatic_joint']}</param>
+                    <param name="initial_value">${initial_state['base_platform_prismatic_joint_position']}</param>
                 </state_interface>
-                <state_interface name="velocity"/>
+                <state_interface name="velocity">
+                    <param name="initial_value">${initial_state['base_platform_prismatic_joint_velocity']}</param>
+                </state_interface>
             </joint>
             <!-- Sensors -->
             <sensor name="lim_switch_neg">
-                <state_interface name="switch_val"/>
+                <state_interface name="switch_val">
+                    <param name="initial_value">${initial_state['lim_switch_neg']}</param>
+                </state_interface>
             </sensor>
-            <sensor name="lim_switch_neg">
-                <state_interface name="swtich_val"/>
+            <sensor name="lim_switch_pos">
+                <state_interface name="swtich_val">
+                    <param name="initial_value">${initial_state['lim_switch_pos']}</param>
+                </state_interface>
             </sensor>
         </ros2_control>

File: linear_slider_description/urdf/linear_slider/linear_slider_macro.xacro (robot description, xacro)
@@ -1,95 +1,97 @@
 <?xml version="1.0" encoding="UTF-8"?>
-<robot name="linear_slider" xmlns:xacro="http://ros.org/wiki/xacro">
-    <!-- ================== -->
-    <!--     Properties     -->
-    <!-- ================== -->
-    <!-- Model properties -->
-    <xacro:property name="ls_frame_mass" value="10.0"/>
-    <xacro:property name="ls_frame_length" value="1.25"/>
-    <xacro:property name="ls_frame_width" value="0.3"/>
-    <xacro:property name="ls_frame_height" value="0.25"/>
-    <xacro:property name="ls_moving_base_mass" value="10.0" />
-    <!-- Model default position/orientation -->
-    <xacro:property name="model_scale" value="0.001 0.001 0.001"/>
-    <xacro:property name="base_link_start_orientation" value="0 0 0"/>
-    <xacro:property name="ls_moving_base_start_orientation" value="0 0 0"/>
-    <xacro:property name="start_offset" value="0.0 0.0 0.0"/>
-    <!-- Prismatic joint properties -->
-    <xacro:property name="slider_limit_min" value="-0.4"/>
-    <xacro:property name="slider_limit_max" value="0.4"/>
-    <xacro:property name="slider_velocity_limit" value="0.25"/>
-    <xacro:property name="slider_effort_limit" value="10"/>
-    <!-- ================== -->
-    <!--     Materials      -->
-    <!-- ================== -->
-    <material name="alpha_black">
-        <color rgba="0.6 0.6 0.6 1"/>
-    </material>
-    <material name="red_v">
-        <color rgba="1 0 0 1"/>
-    </material>
-    <!-- ================== -->
-    <!--       Links        -->
-    <!-- ================== -->
-    <link name="base_link">
-        <visual>
-            <material name="alpha_black"/>
-            <origin rpy="${base_link_start_orientation}" xyz="${start_offset}"/>
-            <geometry>
-                <mesh filename="package://linear_slider_description/meshes/7thlink_fixed.STL" scale="${model_scale}" />
-            </geometry>
-        </visual>
-        <collision>
-            <geometry>
-                <!-- <box size="0.22 0.202 0.118"/> -->
-                <mesh
-                    filename="package://linear_slider_description/meshes/7thlink_fixed.STL"
-                    scale="${model_scale}"
+<robot xmlns:xacro="http://ros.org/wiki/xacro" name="linear_slider">
+    <xacro:macro name="linear_slider" params="prefix">
+        <!-- ================== -->
+        <!--     Properties     -->
+        <!-- ================== -->
+        <!-- Model properties -->
+        <xacro:property name="ls_frame_mass" value="10.0"/>
+        <xacro:property name="ls_frame_length" value="1.25"/>
+        <xacro:property name="ls_frame_width" value="0.3"/>
+        <xacro:property name="ls_frame_height" value="0.25"/>
+        <xacro:property name="ls_moving_base_mass" value="10.0" />
+        <!-- Model default position/orientation -->
+        <xacro:property name="model_scale" value="0.001 0.001 0.001"/>
+        <xacro:property name="base_link_start_orientation" value="0 0 0"/>
+        <xacro:property name="ls_moving_base_start_orientation" value="0 0 0"/>
+        <xacro:property name="start_offset" value="0.0 0.0 0.0"/>
+        <!-- Prismatic joint properties -->
+        <xacro:property name="slider_limit_min" value="-0.4"/>
+        <xacro:property name="slider_limit_max" value="0.4"/>
+        <xacro:property name="slider_velocity_limit" value="0.25"/>
+        <xacro:property name="slider_effort_limit" value="10"/>
+        <!-- ================== -->
+        <!--     Materials      -->
+        <!-- ================== -->
+        <material name="alpha_black">
+            <color rgba="0.6 0.6 0.6 1"/>
+        </material>
+        <material name="red_v">
+            <color rgba="1 0 0 1"/>
+        </material>
+        <!-- ================== -->
+        <!--       Links        -->
+        <!-- ================== -->
+        <link name="${prefix}base_link">
+            <visual>
+                <material name="alpha_black"/>
+                <origin rpy="${base_link_start_orientation}" xyz="${start_offset}"/>
+                <geometry>
+                    <mesh filename="package://linear_slider_description/meshes/7thlink_fixed.STL" scale="${model_scale}" />
+                </geometry>
+            </visual>
+            <collision>
+                <geometry>
+                    <!-- <box size="0.22 0.202 0.118"/> -->
+                    <mesh
+                        filename="package://linear_slider_description/meshes/7thlink_fixed.STL"
+                        scale="${model_scale}"
+                    />
+                </geometry>
+            </collision>
+        </link>
+        <link name="${prefix}ls_moving_base">
+            <visual>
+                <origin rpy="${ls_moving_base_start_orientation}" xyz="${start_offset}" />
+                <material name="red_v" />
+                <geometry>
+                    <mesh
+                        filename="package://linear_slider_description/meshes/7thlink_move.STL"
+                        scale="${model_scale}"
+                    />
+                </geometry>
+            </visual>
+            <collision>
+                <geometry>
+                    <mesh
+                        filename="package://linear_slider_description/meshes/7thlink_move.STL"
+                        scale="${model_scale}" />
+                </geometry>
+            </collision>
+            <inertial>
+                <mass value="${ls_moving_base_mass}" />
+                <origin xyz="0.0 0.0 0.0" />
+                <inertia
+                    ixx="${1*12/(ls_frame_mass + ls_moving_base_mass) * (ls_frame_width**2 + ls_frame_height**2)}"
+                    ixy="0.0"
+                    ixz="0.0"
+                    iyy="${1*12/(ls_frame_mass + ls_moving_base_mass) * (ls_frame_length**2 + ls_frame_height**2)}"
+                    iyz="0.0"
+                    izz="${1*12/(ls_frame_mass + ls_moving_base_mass) * (ls_frame_width**2 + ls_frame_length**2)}"
                 />
-            </geometry>
-        </collision>
-    </link>
-    <link name="ls_moving_base">
-        <visual>
-            <origin rpy="${ls_moving_base_start_orientation}" xyz="${start_offset}" />
-            <material name="red_v" />
-            <geometry>
-                <mesh
-                    filename="package://linear_slider_description/meshes/7thlink_move.STL"
-                    scale="${model_scale}"
-                />
-            </geometry>
-        </visual>
-        <collision>
-            <geometry>
-                <mesh
-                    filename="package://linear_slider_description/meshes/7thlink_move.STL"
-                    scale="${model_scale}" />
-            </geometry>
-        </collision>
-        <inertial>
-            <mass value="${ls_moving_base_mass}" />
-            <origin xyz="0.0 0.0 0.0" />
-            <inertia
-                ixx="${1*12/(ls_frame_mass + ls_moving_base_mass) * (ls_frame_width**2 + ls_frame_height**2)}"
-                ixy="0.0"
-                ixz="0.0"
-                iyy="${1*12/(ls_frame_mass + ls_moving_base_mass) * (ls_frame_length**2 + ls_frame_height**2)}"
-                iyz="0.0"
-                izz="${1*12/(ls_frame_mass + ls_moving_base_mass) * (ls_frame_width**2 + ls_frame_length**2)}"
-            />
-        </inertial>
-    </link>
-        <joint name="base_platform_prismatic_joint" type="prismatic">
-            <parent link="base_link"/>
-            <child link="ls_moving_base"/>
-            <axis xyz="1 0 0"/>
-            <limit
-                effort="${slider_effort_limit}"
-                lower="${slider_limit_min}"
-                upper="${slider_limit_max}"
-                velocity="${slider_velocity_limit}"
-            /> <!-- effort is attribute for enforcing maximum joint effort, between 0 and 100% -->
-            <origin xyz="0.0 0.0 0.0" /> <!-- Define where the joint will be located, defined in terms of parent's reference frame -->
-        </joint>
+            </inertial>
+        </link>
+            <joint name="${prefix}base_platform_prismatic_joint" type="prismatic">
+                <parent link="base_link"/>
+                <child link="ls_moving_base"/>
+                <axis xyz="1 0 0"/>
+                <limit
+                    effort="${slider_effort_limit}"
+                    lower="${slider_limit_min}"
+                    upper="${slider_limit_max}"
+                    velocity="${slider_velocity_limit}"
+                /> <!-- effort is attribute for enforcing maximum joint effort, between 0 and 100% -->
+                <origin xyz="0.0 0.0 0.0" /> <!-- Define where the joint will be located, defined in terms of parent's reference frame -->
+            </joint>
+    </xacro:macro>
 </robot>

File: linear_slider_moveit/config/linear_slider.ros2_control.xacro (robot description, xacro)
@@ -1,5 +1,5 @@
 <?xml version="1.0"?>
 <robot xmlns:xacro="http://www.ros.org/wiki/xacro">
-    <xacro:macro name="linear_slider_ros2_control" params="name initial_positions_file">
+    <xacro:macro name="linear_slider_ros2_control" params="name initial_state_file">
         <xacro:property name="initial_positions" value="${load_yaml(initial_positions_file)['initial_positions']}"/>
         <ros2_control name="${name}" type="system">
