Commit message: fucked up the urdf

File: linear_slider_description/urdf/linear_slider/linear_slider_velocity.ros2_control.xacro (robot description, xacro)
@@ -1,25 +1,30 @@
 <?xml version="1.0"?>
 <robot xmlns:xacro="http://www.ros.org/wiki/xacro">
-    <xacro:macro name="linear_slider_ros2_control" params="name prefix initial_state_file use_mock_hardware:=^|false mock_sensor_commands:=^|false">
+    <xacro:macro name="linear_slider_ros2_control" params="name prefix initial_state_file use_sim:=^|false use_mock_hardware:=^|false mock_sensor_commands:=^|false">
         <xacro:property name="initial_state" value="${xacro.load_yaml(initial_state_file)['initial_state']}"/>
         <ros2_control name="${name}" type="system">
             <!-- Hardware -->
-            <hardware>
-                <!-- By default, set up controllers for simulation. This won't work on real hardware -->
-                <plugin>mock_components/GenericSystem</plugin>
-                <param name="mock_sensor_commands">${mock_sensor_commands}</param>
-                <plugin>linear_slider_system_interface/LinearSliderSystemInterface</plugin>
-                <param name="device_name">linear_slider_ros2_control</param>
-                <param name="joint_name">prismatic_joint</param>
-                <param name="robot_ip">169.254.97.178</param>
-                <!-- <plugin>gz_ros2_control/GazeboSimSystem</plugin> -->
-            </hardware>
+            <xacro:if value="$(arg use_sim)">
+                <hardware>
+                    <plugin>gazebo_ros2_control/GazeboSystem</plugin>
+                </hardware>
+            </xacro:if>
+            <!-- <xacro:unless value="$(arg use_sim)">
+                <hardware>
+                    <param name="device_name">linear_slider_ros2_control</param>
+                    <param name="joint_name">prismatic_joint</param>
+                    <param name="robot_ip">169.254.97.178</param>
+                    <xacro:if value="$(arg use_mock_hardware)">
+                        <plugin>mock_components/GenericSystem</plugin>
+                        <param name="mock_sensor_commands">${mock_sensor_commands}</param>
+                    </xacro:if>
+                    <xacro:unless value="$(arg use_mock_hardware)">
+                        <plugin>linear_slider_system_interface/LinearSliderSystemInterface</plugin>
+                    </xacro:unless>
+                </hardware>
+            </xacro:unless> -->
             <!-- Joints -->
             <joint name="${prefix}joint1">
                 <!-- Command interface -->
-                <command_interface name="position">
-                    <param name="min">-0.40</param>
-                    <param name="max">0.04</param>
-                </command_interface>
                 <command_interface name="velocity">
                     <param name="min">-0.1</param>
@@ -49,7 +54,13 @@
             <plugin filename="libgazebo_ros2_control.so" name="gazebo_ros2_control">
                 <!-- <robot_param>robot_description</robot_param> -->
-                <!-- <robot_param_node>robot_state_publisher<robot_param_node> -->
-                <parameters>$(find linear_slider_bringup)/config/linear_slider_controllers.yaml</parameters>
+                <!-- <robot_param_node>robot_state_publisher</robot_param_node> -->
+                <parameters>$(find linear_slider_bringup)/config/linear_slider_velocity_controller.yaml</parameters>
             </plugin>
+            <sensor name="lim_switch_neg">
+                <always_on>1</always_on>
+            </sensor>
+            <sensor name="lim_switch_pos">
+                <always_on>1</always_on>
+            </sensor>
         </gazebo>
     </xacro:macro>

File: linear_slider_description/urdf/linear_slider_velocity.urdf.xacro (robot description, xacro)
@@ -2,4 +2,5 @@
 <robot xmlns:xacro="http://wiki.ros.org/xacro" name="linear_slider">
     <!-- Use this if parameters are set from the launch file, otherwise delete -->
+    <xacro:arg name="use_sim" default="false" />
     <xacro:arg name="use_mock_hardware" default="false" />
     <xacro:arg name="mock_sensor_commands" default="false" />
@@ -7,5 +8,5 @@
     <!-- Robot description -->
     <xacro:include filename="$(find linear_slider_description)/urdf/linear_slider/linear_slider_macro.xacro"/>
-    <xacro:include filename="$(find linear_slider_description)/urdf/linear_slider/linear_slider.ros2_control.xacro"/>
+    <xacro:include filename="$(find linear_slider_description)/urdf/linear_slider/linear_slider_velocity.ros2_control.xacro"/>
     <xacro:linear_slider_macro prefix="$(arg prefix)" />
     <!-- ros2_control -->
@@ -14,4 +15,5 @@
         prefix="$(arg prefix)"
         initial_state_file="$(find linear_slider_description)/config/initial_state.yaml"
+        use_sim="$(arg use_sim)"
         use_mock_hardware="$(arg use_mock_hardware)"
         mock_sensor_commands="$(arg mock_sensor_commands)"
