Commit message: turns out rviz works better on ubuntu who knew

File: linear_slider_description/urdf/linear_slider/linear_slider.ros2_control.xacro (robot description, xacro)
@@ -15,5 +15,5 @@
             </hardware>
             <!-- Joints -->
-            <joint name="base_platform_prismatic_joint">
+            <joint name="${prefix}base_platform_prismatic_joint">
                 <!-- Command interface -->
                 <command_interface name="position">

Commit message: got a working controller_manager! what a silly api

File: linear_slider_description/urdf/linear_slider/linear_slider.ros2_control.xacro (robot description, xacro)
@@ -6,8 +6,12 @@
             <!-- Hardware -->
             <hardware>
-                <!-- By default, set up controllers for simulation. This won't work on real hardware -->
-                <plugin>mock_components/GenericSystem</plugin>
-                <param name="mock_sensor_commands">${mock_sensor_commands}</param>
-                <plugin>linear_slider_system_interface/LinearSliderSystemInterface</plugin>
+                <xacro:if value="${use_mock_hardware}">
+                    <plugin>mock_components/GenericSystem</plugin>
+                    <param name="mock_sensor_commands">${mock_sensor_commands}</param>
+                </xacro:if>
+                <xacro:unless value="${use_mock_hardware}">
+                    <plugin>linear_slider_hardware_interface/LinearSliderHardwareInterface</plugin>
+                </xacro:unless>
+                <!-- <plugin>linear_slider_system_interface/LinearSliderSystemInterface</plugin> -->
                 <param name="device_name">linear_slider_ros2_control</param>
                 <param name="joint_name">prismatic_joint</param>
@@ -20,5 +24,5 @@
                 <command_interface name="position">
                     <param name="min">-0.40</param>
-                    <param name="max">0.04</param>
+                    <param name="max">0.40</param>
                 </command_interface>
                 <command_interface name="velocity">
@@ -48,6 +52,6 @@
         <gazebo>
             <plugin filename="libgazebo_ros2_control.so" name="gazebo_ros2_control">
-                <!-- <robot_param>robot_description</robot_param> -->
-                <!-- <robot_param_node>robot_state_publisher<robot_param_node> -->
+                <robot_param>robot_description</robot_param>
+                <robot_param_node>robot_state_publisher</robot_param_node>
                 <parameters>$(find linear_slider_bringup)/config/linear_slider_controllers.yaml</parameters>
             </plugin>

File: linear_slider_description/urdf/linear_slider/linear_slider_macro.xacro (robot description, xacro)
@@ -33,4 +33,5 @@
         <!--       Links        -->
         <!-- ================== -->
+        <!-- <link name="world" /> -->
         <link name="${prefix}base_link">
             <visual>

File: linear_slider_description/urdf/linear_slider/linear_slider_velocity.ros2_control.xacro (robot description, xacro)
@@ -1,27 +1,21 @@
 <?xml version="1.0"?>
 <robot xmlns:xacro="http://www.ros.org/wiki/xacro">
-    <xacro:macro name="linear_slider_ros2_control" params="name prefix initial_state_file use_sim:=^|false use_mock_hardware:=^|false mock_sensor_commands:=^|false">
+    <xacro:macro name="linear_slider_ros2_control" params="name prefix initial_state_file use_sim:=^|false use_mock_hardware:=^|false mock_sensor_commands:=^|false"> <!-- The caret ^ indicates to use the outer-scope property (with same name). The pipe | indicates to use the given fallback if the property is not defined in outer scope. -->
         <xacro:property name="initial_state" value="${xacro.load_yaml(initial_state_file)['initial_state']}"/>
         <ros2_control name="${name}" type="system">
             <!-- Hardware -->
-            <xacro:if value="$(arg use_sim)">
-                <hardware>
+            <hardware>
+                <xacro:if value="${use_mock_hardware}">
+                    <plugin>mock_components/GenericSystem</plugin>
+                </xacro:if>
+                <xacro:unless value="${use_mock_hardware}">
                     <plugin>gazebo_ros2_control/GazeboSystem</plugin>
-                </hardware>
-            </xacro:if>
-            <!-- <xacro:unless value="$(arg use_sim)">
-                <hardware>
-                    <param name="device_name">linear_slider_ros2_control</param>
-                    <param name="joint_name">prismatic_joint</param>
-                    <param name="robot_ip">169.254.97.178</param>
-                    <xacro:if value="$(arg use_mock_hardware)">
-                        <plugin>mock_components/GenericSystem</plugin>
-                        <param name="mock_sensor_commands">${mock_sensor_commands}</param>
-                    </xacro:if>
-                    <xacro:unless value="$(arg use_mock_hardware)">
-                        <plugin>linear_slider_system_interface/LinearSliderSystemInterface</plugin>
-                    </xacro:unless>
-                </hardware>
-            </xacro:unless> -->
+                </xacro:unless>
+                <param name="mock_sensor_commands">${mock_sensor_commands}</param>
+                <!-- <plugin>linear_slider_system_interface/LinearSliderSystemInterface</plugin> -->
+                <param name="device_name">linear_slider_ros2_control</param>
+                <param name="joint_name">prismatic_joint</param>
+                <param name="robot_ip">169.254.97.178</param>
+            </hardware>
             <!-- Joints -->
             <joint name="${prefix}joint1">
@@ -46,22 +40,33 @@
             </sensor>
             <sensor name="lim_switch_pos">
-                <state_interface name="swtich_val">
+                <state_interface name="switch_val">
                     <param name="initial_value">${initial_state['lim_switch_pos']}</param>
                 </state_interface>
             </sensor>
         </ros2_control>
-        <gazebo>
-            <plugin filename="libgazebo_ros2_control.so" name="gazebo_ros2_control">
-                <!-- <robot_param>robot_description</robot_param> -->
-                <!-- <robot_param_node>robot_state_publisher</robot_param_node> -->
-                <parameters>$(find linear_slider_bringup)/config/linear_slider_velocity_controller.yaml</parameters>
-            </plugin>
-            <sensor name="lim_switch_neg">
-                <always_on>1</always_on>
-            </sensor>
-            <sensor name="lim_switch_pos">
-                <always_on>1</always_on>
-            </sensor>
-        </gazebo>
+        <!-- Gazebo -->
+        <xacro:unless value="${use_mock_hardware}">
+            <gazebo>
+                <plugin filename="libgazebo_ros2_control.so" name="gazebo_ros2_control">
+                    <!-- <robotNamespace>/linear_slider</robotNamespace> -->
+                    <robot_param>robot_description</robot_param>
+                    <robot_param_node>robot_state_publisher</robot_param_node>
+                    <parameters>$(find linear_slider_bringup)/config/linear_slider_velocity_controller.yaml</parameters>
+                </plugin>
+                <sensor name="lim_switch_neg">
+                    <always_on>1</always_on>
+                </sensor>
+                <sensor name="lim_switch_pos">
+                    <always_on>1</always_on>
+                </sensor>
+            </gazebo>
+            <gazebo reference="${prefix}base_link">
+                <material>Gazebo/Gray</material>
+            </gazebo>
+            <gazebo reference="${prefix}joint1"/>
+            <gazebo reference="${prefix}moving_base">
+                <material>Gazebo/Red</material>
+            </gazebo>
+        </xacro:unless>
     </xacro:macro>
 </robot>

File: linear_slider_description/urdf/linear_slider_velocity.urdf.xacro (robot description, xacro)
@@ -3,5 +3,5 @@
     <!-- Use this if parameters are set from the launch file, otherwise delete -->
     <xacro:arg name="use_sim" default="false" />
-    <xacro:arg name="use_mock_hardware" default="false" />
+    <xacro:arg name="use_mock_hardware" default="true" />
     <xacro:arg name="mock_sensor_commands" default="false" />
     <xacro:arg name="prefix" default="''" />
@@ -12,5 +12,5 @@
     <!-- ros2_control -->
     <xacro:linear_slider_ros2_control
-        name="linear_slider"
+        name="linear_slider_ros2_control"
         prefix="$(arg prefix)"
         initial_state_file="$(find linear_slider_description)/config/initial_state.yaml"
