Commit message: updates to moveit config package, goal executed but rviz not moving. mock_hardware/GenericSystem problem?

File: linear_slider_description/urdf/linear_slider/linear_slider_macro.xacro (robot description, xacro)
@@ -21,5 +21,5 @@
         <xacro:property name="slider_limit_max" value="0.4"/>
         <xacro:property name="slider_velocity_limit" value="0.25"/>
-        <xacro:property name="slider_effort_limit" value="10"/>
+        <xacro:property name="slider_effort_limit" value="2"/>
         <!-- tool0 / flange properties -->
         <xacro:property name="moving_base__flange_offset" value="0.05" />

File: linear_slider_moveit_config/srdf/linear_slider.srdf.xacro (robot description, xacro)
@@ -7,5 +7,5 @@
     <xacro:arg name="prefix" default=""/>
     <xacro:arg name="name" default="linear_slider"/>
-    <xacro:include filename="$(find linear_slider_moveit)/srdf/linear_slider_macro.srdf.xacro"/>
+    <xacro:include filename="$(find linear_slider_moveit_config)/srdf/linear_slider_macro.srdf.xacro"/>
     <xacro:linear_slider_srdf name="$(arg name)" prefix="$(arg prefix)" />
 </robot>
