Commit message: decided to get a working moveit for just the linear slider first. Made some updates in this direction

File: linear_slider_moveit/config/ur_with_linear_slider.ros2_control.xacro (robot description, xacro)
@@ -1,5 +1,5 @@
 <?xml version="1.0"?>
 <robot xmlns:xacro="http://www.ros.org/wiki/xacro">
-    <xacro:macro name="linear_slider_ros2_control" params="name initial_positions_file">
+    <xacro:macro name="ur_with_linear_slider_ros2_control" params="name initial_positions_file">
         <xacro:property name="initial_positions" value="${load_yaml(initial_positions_file)['initial_positions']}"/>
         <ros2_control name="${name}" type="system">
@@ -8,8 +8,8 @@
                 <plugin>mock_components/GenericSystem</plugin>
             </hardware>
-            <joint name="joint1">
+            <joint name="linear_slider/joint1">
                 <command_interface name="velocity"/>
                 <state_interface name="position">
-                  <param name="initial_value">${initial_positions['joint1']}</param>
+                  <param name="initial_value">${initial_positions['linear_slider/joint1']}</param>
                 </state_interface>
                 <state_interface name="velocity"/>
