Commit message: changed a joint name. Still need to fix bringup package for controller default parameters

File: linear_slider_description/urdf/linear_slider.urdf (robot description, URDF)
Before this commit: robot linear_slider, 2 links, 1 joints
Links:
- removed link ls_moving_base
- added link moving_base, mass 10.0; collision mesh filename=package://linear_slider_description/meshes/7thlink_move.STL scale=0.001 0.001 0.001; visual mesh filename=package://linear_slider_description/meshes/7thlink_move.STL scale=0.001 0.001 0.001
Joints:
- removed joint base_platform_prismatic_joint
- added joint joint1: type prismatic, parent base_link, child moving_base, origin xyz=0.0 0.0 0.0, axis 1 0 0, limit lower=-0.4 upper=0.4 effort=10 velocity=0.25

File: linear_slider_description/urdf/linear_slider/linear_slider.ros2_control.xacro (robot description, xacro)
@@ -15,5 +15,5 @@
             </hardware>
             <!-- Joints -->
-            <joint name="${prefix}base_platform_prismatic_joint">
+            <joint name="${prefix}joint1">
                 <!-- Command interface -->
                 <command_interface name="position">
@@ -27,8 +27,8 @@
                 <!-- State interface -->
                 <state_interface name="position">
-                    <param name="initial_value">${initial_state['base_platform_prismatic_joint_position']}</param>
+                    <param name="initial_value">${initial_state['joint1_position']}</param>
                 </state_interface>
                 <state_interface name="velocity">
-                    <param name="initial_value">${initial_state['base_platform_prismatic_joint_velocity']}</param>
+                    <param name="initial_value">${initial_state['joint1_velocity']}</param>
                 </state_interface>
             </joint>

File: linear_slider_description/urdf/linear_slider/linear_slider_macro.xacro (robot description, xacro)
@@ -6,13 +6,13 @@
         <!-- ================== -->
         <!-- Model properties -->
-        <xacro:property name="ls_frame_mass" value="10.0"/>
-        <xacro:property name="ls_frame_length" value="1.25"/>
-        <xacro:property name="ls_frame_width" value="0.3"/>
-        <xacro:property name="ls_frame_height" value="0.25"/>
-        <xacro:property name="ls_moving_base_mass" value="10.0" />
+        <xacro:property name="frame_mass" value="10.0"/>
+        <xacro:property name="frame_length" value="1.25"/>
+        <xacro:property name="frame_width" value="0.3"/>
+        <xacro:property name="frame_height" value="0.25"/>
+        <xacro:property name="moving_base_mass" value="10.0" />
         <!-- Model default position/orientation -->
         <xacro:property name="model_scale" value="0.001 0.001 0.001"/>
         <xacro:property name="base_link_start_orientation" value="0 0 0"/>
-        <xacro:property name="ls_moving_base_start_orientation" value="0 0 0"/>
+        <xacro:property name="moving_base_start_orientation" value="0 0 0"/>
         <xacro:property name="start_offset" value="0.0 0.0 0.0"/>
         <!-- Prismatic joint properties -->
@@ -51,7 +51,7 @@
             </collision>
         </link>
-        <link name="${prefix}ls_moving_base">
+        <link name="${prefix}moving_base">
             <visual>
-                <origin rpy="${ls_moving_base_start_orientation}" xyz="${start_offset}" />
+                <origin rpy="${moving_base_start_orientation}" xyz="${start_offset}" />
                 <material name="red_v" />
                 <geometry>
@@ -70,19 +70,19 @@
             </collision>
             <inertial>
-                <mass value="${ls_moving_base_mass}" />
+                <mass value="${moving_base_mass}" />
                 <origin xyz="0.0 0.0 0.0" />
                 <inertia
-                    ixx="${1*12/(ls_frame_mass + ls_moving_base_mass) * (ls_frame_width**2 + ls_frame_height**2)}"
+                    ixx="${1*12/(frame_mass + moving_base_mass) * (frame_width**2 + frame_height**2)}"
                     ixy="0.0"
                     ixz="0.0"
-                    iyy="${1*12/(ls_frame_mass + ls_moving_base_mass) * (ls_frame_length**2 + ls_frame_height**2)}"
+                    iyy="${1*12/(frame_mass + moving_base_mass) * (frame_length**2 + frame_height**2)}"
                     iyz="0.0"
-                    izz="${1*12/(ls_frame_mass + ls_moving_base_mass) * (ls_frame_width**2 + ls_frame_length**2)}"
+                    izz="${1*12/(frame_mass + moving_base_mass) * (frame_width**2 + frame_length**2)}"
                 />
             </inertial>
         </link>
-            <joint name="${prefix}base_platform_prismatic_joint" type="prismatic">
+            <joint name="${prefix}joint1" type="prismatic">
                 <parent link="base_link"/>
-                <child link="ls_moving_base"/>
+                <child link="moving_base"/>
                 <axis xyz="1 0 0"/>
                 <limit

File: linear_slider_moveit/config/linear_slider.ros2_control.xacro (robot description, xacro)
@@ -8,9 +8,9 @@
                 <plugin>mock_components/GenericSystem</plugin>
             </hardware>
-            <joint name="base_platform_prismatic_joint">
+            <joint name="joint1">
                 <command_interface name="position"/>
                 <command_interface name="velocity"/>
                 <state_interface name="position">
-                  <param name="initial_value">${initial_positions['base_platform_prismatic_joint']}</param>
+                  <param name="initial_value">${initial_positions['joint1']}</param>
                 </state_interface>
                 <state_interface name="velocity"/>

Commit message: add gazebo sim, but it doesn't like something about the interface, probably with the URDF

File: linear_slider_description/urdf/linear_slider.urdf (robot description, URDF)
Before this commit: robot linear_slider, 2 links, 1 joints
Links:
- added link world
- link base_link: geometry collision box size=0.8 0.3 0.14; visual mesh filename=package://linear_slider_description/meshes/7thlink_fixed.STL scale=0.001 0.001 0.001
- link moving_base: geometry collision box size=0.22 0.202 0.118; visual mesh filename=package://linear_slider_description/meshes/7thlink_move.STL scale=0.001 0.001 0.001
Joints:
- added joint base_joint: type fixed, parent world, child base_link, origin xyz=0 0 0 rpy=0 0 0

File: linear_slider_description/urdf/linear_slider.urdf.xacro (robot description, xacro)
@@ -2,18 +2,66 @@
 <robot xmlns:xacro="http://wiki.ros.org/xacro" name="linear_slider">
     <!-- Use this if parameters are set from the launch file, otherwise delete -->
+    <xacro:arg name="prefix" default="''" />
     <xacro:arg name="use_mock_hardware" default="false" />
     <xacro:arg name="mock_sensor_commands" default="false" />
-    <xacro:arg name="prefix" default="''" />
+    <xacro:arg name="sim_gazebo" default="false" />
+    <xacro:arg name="sim_gazebo_classic" default="false"/>
+    <!-- <xacro:arg name="simulation_controllers" default="" /> -->
     <!-- Robot description -->
     <xacro:include filename="$(find linear_slider_description)/urdf/linear_slider/linear_slider_macro.xacro"/>
     <xacro:include filename="$(find linear_slider_description)/urdf/linear_slider/linear_slider.ros2_control.xacro"/>
-    <xacro:linear_slider_macro prefix="$(arg prefix)" />
+    <!-- World link -->
+    <link name="world" />
+    <xacro:linear_slider_macro prefix="$(arg prefix)" parent="world">
+        <origin xyz="0 0 0" rpy="0 0 0"/>
+    </xacro:linear_slider_macro>
     <!-- ros2_control -->
     <xacro:linear_slider_ros2_control
-        name="linear_slider"
+        name="linear_slider_ros2_control"
         prefix="$(arg prefix)"
         initial_state_file="$(find linear_slider_description)/config/initial_state.yaml"
+        sim_gazebo="$(arg sim_gazebo)"
+        sim_gazebo_classic="$(arg sim_gazebo_classic)"
         use_mock_hardware="$(arg use_mock_hardware)"
         mock_sensor_commands="$(arg mock_sensor_commands)"
     />
+    <xacro:if value="$(arg sim_gazebo_classic)">
+        <!-- ================== -->
+        <!--   Gazebo Classic   -->
+        <!-- ================== -->
+        <gazebo reference="world"/>
+        <gazebo>
+            <plugin filename="libgazebo_ros2_control.so" name="gazebo_ros2_control">
+                <robot_param>robot_description</robot_param>
+                <robot_param_node>robot_state_publisher</robot_param_node>
+                <parameters>$(find linear_slider_bringup)/config/linear_slider_controllers.yaml</parameters>
+                <!-- <parameters>$(arg simulation_controllers)</parameters> -->
+            </plugin>
+            <!-- <sensor name="lim_switch_neg">
+                <always_on>1</always_on>
+            </sensor>
+            <sensor name="lim_switch_pos">
+                <always_on>1</always_on>
+            </sensor> -->
+        </gazebo>
+        <gazebo reference="$(arg prefix)joint1"/>
+        <gazebo reference="$(arg prefix)base_link">
+            <material>Gazebo/Gray</material>
+        </gazebo>
+        <gazebo reference="$(arg prefix)moving_base">
+            <material>Gazebo/Red</material>
+        </gazebo>
+    </xacro:if>
+    <xacro:if value="$(arg sim_gazebo)">
+        <!-- ================== -->
+        <!--  Gazebo Ignition   -->
+        <!-- ================== -->
+        <gazebo reference="world"/>
+        <gazebo>
+            <plugin filename="libign_ros2_control-system.so" name="ign_ros2_control::IgnitionROS2ControlPlugin">
+                <parameters>$(find linear_slider_bringup)/config/linear_slider_controllers.yaml</parameters>
+                <controller_manager_node_name>$(arg prefix)controller_manager</controller_manager_node_name>
+            </plugin>
+        </gazebo>
+    </xacro:if>
 </robot>

File: linear_slider_description/urdf/linear_slider/linear_slider.ros2_control.xacro (robot description, xacro)
@@ -1,6 +1,17 @@
 <?xml version="1.0"?>
 <robot xmlns:xacro="http://www.ros.org/wiki/xacro">
-    <xacro:macro name="linear_slider_ros2_control" params="name prefix initial_state_file use_mock_hardware:=^|false mock_sensor_commands:=^|false">
+    <xacro:macro name="linear_slider_ros2_control" params="
+        name
+        prefix
+        initial_state_file
+        sim_gazebo:=^|false
+        sim_gazebo_classic:=^|false
+        use_mock_hardware:=^|false
+        mock_sensor_commands:=^|false"
+        > <!-- The caret ^ indicates to use the outer-scope property (with same name). The pipe | indicates to use the given fallback if the property is not defined in outer scope. -->
         <xacro:property name="initial_state" value="${xacro.load_yaml(initial_state_file)['initial_state']}"/>
+        <!-- ================== -->
+        <!--    ros2_control    -->
+        <!-- ================== -->
         <ros2_control name="${name}" type="system">
             <!-- Hardware -->
@@ -10,12 +21,16 @@
                     <param name="mock_sensor_commands">${mock_sensor_commands}</param>
                 </xacro:if>
-                <xacro:unless value="${use_mock_hardware}">
+                <xacro:if value="${sim_gazebo_classic}">
+                    <plugin>gazebo_ros2_control/GazeboSystem</plugin>
+                </xacro:if>
+                <xacro:if value="${sim_gazebo}">
+                    <plugin>ign_ros2_control/IgnitionSystem</plugin>
+                </xacro:if>
+                <xacro:unless value="${use_mock_hardware or sim_gazebo or sim_gazebo_classic}">
                     <plugin>linear_slider_hardware_interface/LinearSliderHardwareInterface</plugin>
                 </xacro:unless>
-                <!-- <plugin>linear_slider_system_interface/LinearSliderSystemInterface</plugin> -->
-                <param name="device_name">linear_slider_ros2_control</param>
+                <!-- <param name="device_name">linear_slider_device</param>
                 <param name="joint_name">prismatic_joint</param>
-                <param name="robot_ip">169.254.97.178</param>
-                <!-- <plugin>gz_ros2_control/GazeboSimSystem</plugin> -->
+                <param name="robot_ip">169.254.97.178</param> -->
             </hardware>
             <!-- Joints -->
@@ -26,18 +41,18 @@
                     <param name="max">0.40</param>
                 </command_interface>
-                <command_interface name="velocity">
+                <!-- <command_interface name="velocity">
                     <param name="min">-0.1</param>
                     <param name="max">0.1</param>
-                </command_interface>
+                </command_interface> -->
                 <!-- State interface -->
                 <state_interface name="position">
                     <param name="initial_value">${initial_state['joint1_position']}</param>
                 </state_interface>
-                <state_interface name="velocity">
+                <!-- <state_interface name="velocity">
                     <param name="initial_value">${initial_state['joint1_velocity']}</param>
-                </state_interface>
+                </state_interface> -->
             </joint>
             <!-- Sensors -->
-            <sensor name="lim_switch_neg">
+            <!-- <sensor name="lim_switch_neg">
                 <state_interface name="switch_val">
                     <param name="initial_value">${initial_state['lim_switch_neg']}</param>
@@ -45,16 +60,9 @@
             </sensor>
             <sensor name="lim_switch_pos">
-                <state_interface name="swtich_val">
+                <state_interface name="switch_val">
                     <param name="initial_value">${initial_state['lim_switch_pos']}</param>
                 </state_interface>
-            </sensor>
+            </sensor> -->
         </ros2_control>
-        <gazebo>
-            <plugin filename="libgazebo_ros2_control.so" name="gazebo_ros2_control">
-                <robot_param>robot_description</robot_param>
-                <robot_param_node>robot_state_publisher</robot_param_node>
-                <parameters>$(find linear_slider_bringup)/config/linear_slider_controllers.yaml</parameters>
-            </plugin>
-        </gazebo>
     </xacro:macro>
 </robot>

File: linear_slider_description/urdf/linear_slider/linear_slider_macro.xacro (robot description, xacro)
@@ -1,5 +1,5 @@
 <?xml version="1.0" encoding="UTF-8"?>
 <robot xmlns:xacro="http://ros.org/wiki/xacro" name="linear_slider">
-    <xacro:macro name="linear_slider_macro" params="prefix">
+    <xacro:macro name="linear_slider_macro" params="prefix parent *origin">
         <!-- ================== -->
         <!--     Properties     -->
@@ -33,5 +33,4 @@
         <!--       Links        -->
         <!-- ================== -->
-        <!-- <link name="world" /> -->
         <link name="${prefix}base_link">
             <visual>
@@ -44,9 +43,9 @@
             <collision>
                 <geometry>
-                    <!-- <box size="0.22 0.202 0.118"/> -->
-                    <mesh
+                    <box size="1.0 0.3 0.10"/>
+                    <!-- <mesh
                         filename="package://linear_slider_description/meshes/7thlink_fixed.STL"
                         scale="${model_scale}"
-                    />
+                    /> -->
                 </geometry>
             </collision>
@@ -65,7 +64,9 @@
             <collision>
                 <geometry>
-                    <mesh
+                    <box size="0.22 0.202 0.118"/>
+                    <!-- <mesh
                         filename="package://linear_slider_description/meshes/7thlink_move.STL"
-                        scale="${model_scale}" />
+                        scale="${model_scale}"
+                    /> -->
                 </geometry>
             </collision>
@@ -83,16 +84,24 @@
             </inertial>
         </link>
-            <joint name="${prefix}joint1" type="prismatic">
-                <parent link="base_link"/>
-                <child link="moving_base"/>
-                <axis xyz="1 0 0"/>
-                <limit
-                    effort="${slider_effort_limit}"
-                    lower="${slider_limit_min}"
-                    upper="${slider_limit_max}"
-                    velocity="${slider_velocity_limit}"
-                /> <!-- effort is attribute for enforcing maximum joint effort, between 0 and 100% -->
-                <origin xyz="0.0 0.0 0.0" /> <!-- Define where the joint will be located, defined in terms of parent's reference frame -->
-            </joint>
+        <!-- ================== -->
+        <!--       Joints       -->
+        <!-- ================== -->
+        <joint name="${prefix}base_joint" type="fixed">
+            <parent link="${parent}"/>
+            <child link="${prefix}base_link"/>
+            <xacro:insert_block name="origin"/>
+        </joint>
+        <joint name="${prefix}joint1" type="prismatic">
+            <parent link="base_link"/>
+            <child link="moving_base"/>
+            <axis xyz="1 0 0"/>
+            <limit
+                effort="${slider_effort_limit}"
+                lower="${slider_limit_min}"
+                upper="${slider_limit_max}"
+                velocity="${slider_velocity_limit}"
+            /> <!-- effort is attribute for enforcing maximum joint effort, between 0 and 100% -->
+            <origin xyz="0.0 0.0 0.0" /> <!-- Define where the joint will be located, defined in terms of parent's reference frame -->
+        </joint>
     </xacro:macro>
 </robot>

File: linear_slider_moveit/config/linear_slider.ros2_control.xacro (robot description, xacro)
@@ -1,5 +1,5 @@
 <?xml version="1.0"?>
 <robot xmlns:xacro="http://www.ros.org/wiki/xacro">
-    <xacro:macro name="linear_slider_ros2_control" params="name initial_state_file">
+    <xacro:macro name="linear_slider_ros2_control" params="name initial_positions_file">
         <xacro:property name="initial_positions" value="${load_yaml(initial_positions_file)['initial_positions']}"/>
         <ros2_control name="${name}" type="system">
@@ -10,9 +10,7 @@
             <joint name="joint1">
                 <command_interface name="position"/>
-                <command_interface name="velocity"/>
                 <state_interface name="position">
                   <param name="initial_value">${initial_positions['joint1']}</param>
                 </state_interface>
-                <state_interface name="velocity"/>
             </joint>
         </ros2_control>

File: linear_slider_moveit/config/linear_slider.urdf.xacro (robot description, xacro)
@@ -3,5 +3,5 @@
     <xacro:arg name="initial_positions_file" default="initial_positions.yaml" />
     <!-- Import linear_slider urdf file -->
-    <xacro:include filename="$(find linear_slider_description)/urdf/linear_slider.urdf" />
+    <xacro:include filename="$(find linear_slider_description)/urdf/linear_slider.urdf.xacro" />
     <!-- Import control_xacro -->
     <xacro:include filename="linear_slider.ros2_control.xacro" />
