Commit message: Updated READMEs for each package for final project submission

File: linear_slider_description/urdf/linear_slider.urdf (robot description, URDF)
Before this commit: robot linear_slider, 3 links, 2 joints
Links:
- added link base
- added link flange
- added link tool0
- link base_link: geometry collision box size=1.0 0.3 0.10; visual mesh filename=package://linear_slider_description/meshes/7thlink_fixed.STL scale=0.001 0.001 0.001
Joints:
- added joint base_link-base_joint: type fixed, parent base_link, child base, origin xyz=0 0 0 rpy=0 0 0
- added joint moving_base-tool0: type fixed, parent moving_base, child tool0, origin xyz=0 0 0 rpy=0 0 0
- added joint tool0-flange_joint: type fixed, parent tool0, child flange, origin xyz=0 0 0 rpy=0 0 0

File: linear_slider_description/urdf/linear_slider.urdf.xacro (robot description, xacro)
@@ -13,4 +13,5 @@
     <!-- World link -->
     <link name="world" />
+    <!-- Macro information -->
     <xacro:linear_slider_macro prefix="$(arg prefix)" parent="world">
         <origin xyz="0 0 0" rpy="0 0 0"/>
@@ -45,11 +46,4 @@
             </sensor> -->
         </gazebo>
-        <gazebo reference="$(arg prefix)joint1"/>
-        <gazebo reference="$(arg prefix)base_link">
-            <material>Gazebo/Gray</material>
-        </gazebo>
-        <gazebo reference="$(arg prefix)moving_base">
-            <material>Gazebo/Red</material>
-        </gazebo>
     </xacro:if>
     <xacro:if value="$(arg sim_gazebo)">

File: linear_slider_description/urdf/linear_slider/linear_slider.ros2_control.xacro (robot description, xacro)
@@ -54,8 +54,9 @@
             </joint>
             <!-- Sensors -->
-            <!-- <sensor name="lim_switch_neg">
+            <sensor name="lim_switch_neg">
                 <state_interface name="switch_val">
                     <param name="initial_value">${initial_state['lim_switch_neg']}</param>
                 </state_interface>
+                <param name="frame_id">${prefix}base_link</param>
             </sensor>
             <sensor name="lim_switch_pos">
@@ -63,5 +64,6 @@
                     <param name="initial_value">${initial_state['lim_switch_pos']}</param>
                 </state_interface>
-            </sensor> -->
+                <param name="frame_id">${prefix}base_link</param>
+            </sensor>
         </ros2_control>
     </xacro:macro>

File: linear_slider_description/urdf/linear_slider/linear_slider_macro.xacro (robot description, xacro)
@@ -33,4 +33,5 @@
         <!--       Links        -->
         <!-- ================== -->
+        <!-- base_link -->
         <link name="${prefix}base_link">
             <visual>
@@ -51,4 +52,8 @@
             </collision>
         </link>
+        <gazebo reference="${prefix}base_link">
+            <material>Gazebo/Gray</material>
+        </gazebo>
+        <!-- moving_base link -->
         <link name="${prefix}moving_base">
             <visual>
@@ -84,7 +89,16 @@
             </inertial>
         </link>
+        <gazebo reference="${prefix}moving_base">
+            <material>Gazebo/Red</material>
+        </gazebo>
+        <!-- tool link -->
+        <link name="${prefix}tool0" />
+        <link name="${prefix}base" />
+        <!-- Frame for mounting EEF models to a manipulator. x+ axis points forward (REP 103). -->
+        <link name="${prefix}flange" />
         <!-- ================== -->
         <!--       Joints       -->
         <!-- ================== -->
+        <!-- base_joint fixes base_link to the environment -->
         <joint name="${prefix}base_joint" type="fixed">
             <parent link="${parent}"/>
@@ -92,4 +106,5 @@
             <xacro:insert_block name="origin"/>
         </joint>
+        <!-- joint1 -->
         <joint name="${prefix}joint1" type="prismatic">
             <parent link="base_link"/>
@@ -104,4 +119,21 @@
             <origin xyz="0.0 0.0 0.0" /> <!-- Define where the joint will be located, defined in terms of parent's reference frame -->
         </joint>
+        <!-- Extra joints for ros-industrial standard compatability -->
+        <!-- tool frame to fixed frame -->
+        <joint name="${prefix}moving_base-tool0" type="fixed">
+            <parent link="${prefix}moving_base"/>
+            <child link="${prefix}tool0"/>
+            <origin xyz="0 0 0" rpy="0 0 0" />
+        </joint>
+        <joint name="${prefix}base_link-base_joint" type="fixed">
+            <origin xyz="0 0 0" rpy="0 0 0" />
+            <parent link="${prefix}base_link" />
+            <child link="${prefix}base" />
+        </joint>
+        <joint name="${prefix}tool0-flange_joint" type="fixed">
+            <origin xyz="0 0 0" rpy="0 0 0" />
+            <parent link="${prefix}tool0" />
+            <child link="${prefix}flange" />
+        </joint>
     </xacro:macro>
 </robot>

Commit message: added inertial link to base_link

File: linear_slider_description/urdf/linear_slider.urdf (robot description, URDF)
Before this commit: robot linear_slider, 6 links, 5 joints
Links:
- link base_link: mass None -> 1000.0

File: linear_slider_description/urdf/linear_slider/linear_slider_macro.xacro (robot description, xacro)
@@ -51,4 +51,16 @@
                 </geometry>
             </collision>
+            <inertial>
+                <mass value="1000.0" />
+                <origin xyz="0.0 0.0 0.0" />
+                <inertia
+                    ixx="${1*12/(frame_mass + 1000.0) * (frame_width**2 + frame_height**2)}"
+                    ixy="0.0"
+                    ixz="0.0"
+                    iyy="${1*12/(frame_mass + 1000.0) * (frame_length**2 + frame_height**2)}"
+                    iyz="0.0"
+                    izz="${1*12/(frame_mass + 1000.0) * (frame_width**2 + frame_length**2)}"
+                />
+            </inertial>
         </link>
         <gazebo reference="${prefix}base_link">

Commit message: fixed rviz model topic issue

File: linear_slider_description/urdf/linear_slider.urdf (robot description, URDF)
Before this commit: robot linear_slider, 6 links, 5 joints
Links:
- link base_link: mass 1000.0 -> 20.0; geometry collision box size=1.0 0.3 0.10; visual mesh filename=file:///home/main/ros2_ws/install/linear_slider_description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 scale=0.001 0.001 0.001
- link moving_base: geometry collision box size=0.22 0.202 0.118; visual mesh filename=file:///home/main/ros2_ws/install/linear_slider_description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 scale=0.001 0.001 0.001

Commit message: made some changes to the URDF structure, still having TF issues

File: linear_slider_description/urdf/linear_slider.urdf (robot description, URDF)
Before this commit: robot linear_slider, 6 links, 5 joints
Links:
- removed link base
- removed link base_link
- removed link flange
- removed link moving_base
- removed link tool0
- added link linear_slider__base
- added link linear_slider__base_link, mass 20.0; collision box size=1.0 0.3 0.10; visual mesh filename=file:///home/luke/ros2_ws/install/linear_slider_description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 scale=0.001 0.001 0.001
- added link linear_slider__flange
- added link linear_slider__moving_base, mass 10.0; collision box size=0.22 0.202 0.118; visual mesh filename=file:///home/luke/ros2_ws/install/linear_slider_description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 scale=0.001 0.001 0.001
- added link linear_slider__tool0
Joints:
- removed joint base_joint
- removed joint base_link-base_joint
- removed joint joint1
- removed joint moving_base-tool0
- removed joint tool0-flange_joint
- added joint linear_slider__base_joint: type fixed, parent world, child linear_slider__base, origin xyz=0 0 0 rpy=0 0 0
- added joint linear_slider__base_link__base_joint: type fixed, parent linear_slider__base, child linear_slider__base_link, origin xyz=0 0 0 rpy=0 0 0
- added joint linear_slider__flange__tool0_joint: type fixed, parent linear_slider__flange, child linear_slider__tool0, origin xyz=0 0 0 rpy=0 0 0
- added joint linear_slider__joint1: type prismatic, parent linear_slider__base_link, child linear_slider__moving_base, origin xyz=0 0 0 rpy=0 0 0, axis 1 0 0, limit lower=-0.4 upper=0.4 effort=10 velocity=0.25
- added joint linear_slider__moving_base__flange_joint: type fixed, parent linear_slider__moving_base, child linear_slider__flange, origin xyz=0 0 0.05 rpy=0 0 0

File: linear_slider_description/urdf/linear_slider.urdf.xacro (robot description, xacro)
@@ -1,5 +1,6 @@
-<?xml version="1.0" encoding="UTF-8"?>
-<robot xmlns:xacro="http://wiki.ros.org/xacro" name="linear_slider">
-    <!-- Use this if parameters are set from the launch file, otherwise delete -->
+<?xml version="1.0"?>
+<robot xmlns:xacro="https://ros.org/wiki/xacro" name="linear_slider">
+    <!-- linear slider -->
+    <xacro:include filename="$(find linear_slider_description)/urdf/linear_slider_base.urdf.xacro" />
     <xacro:arg name="prefix" default="''" />
     <xacro:arg name="use_mock_hardware" default="false" />
@@ -7,57 +8,10 @@
     <xacro:arg name="sim_gazebo" default="false" />
     <xacro:arg name="sim_gazebo_classic" default="false"/>
-    <!-- <xacro:arg name="simulation_controllers" default="" /> -->
-    <!-- Robot description -->
-    <xacro:include filename="$(find linear_slider_description)/urdf/linear_slider/linear_slider_macro.xacro"/>
-    <xacro:include filename="$(find linear_slider_description)/urdf/linear_slider/linear_slider.ros2_control.xacro"/>
-    <!-- World link -->
-    <link name="world" />
-    <!-- Macro information -->
-    <xacro:linear_slider_macro prefix="$(arg prefix)" parent="world">
-        <origin xyz="0 0 0" rpy="0 0 0"/>
-    </xacro:linear_slider_macro>
-    <!-- ros2_control -->
-    <xacro:linear_slider_ros2_control
-        name="linear_slider_ros2_control"
-        prefix="$(arg prefix)"
-        initial_state_file="$(find linear_slider_description)/config/initial_state.yaml"
-        sim_gazebo="$(arg sim_gazebo)"
-        sim_gazebo_classic="$(arg sim_gazebo_classic)"
-        use_mock_hardware="$(arg use_mock_hardware)"
-        mock_sensor_commands="$(arg mock_sensor_commands)"
+    <xacro:linear_slider
+            prefix="$(arg prefix)"
+            sim_gazebo="$(arg sim_gazebo)"
+            sim_gazebo_classic="$(arg sim_gazebo_classic)"
+            use_mock_hardware="$(arg use_mock_hardware)"
+            mock_sensor_commands="$(arg mock_sensor_commands)"
     />
-    <xacro:if value="$(arg sim_gazebo_classic)">
-        <!-- ================== -->
-        <!--   Gazebo Classic   -->
-        <!-- ================== -->
-        <gazebo reference="$(arg prefix)base_link">
-            <static>true</static>
-        </gazebo>
-        <gazebo>
-            <plugin filename="libgazebo_ros2_control.so" name="gazebo_ros2_control">
-                <robot_param>robot_description</robot_param>
-                <robot_param_node>robot_state_publisher</robot_param_node>
-                <parameters>$(find linear_slider_bringup)/config/linear_slider_controllers.yaml</parameters>
-                <!-- <parameters>$(arg simulation_controllers)</parameters> -->
-            </plugin>
-            <!-- <sensor name="lim_switch_neg">
-                <always_on>1</always_on>
-            </sensor>
-            <sensor name="lim_switch_pos">
-                <always_on>1</always_on>
-            </sensor> -->
-        </gazebo>
-    </xacro:if>
-    <xacro:if value="$(arg sim_gazebo)">
-        <!-- ================== -->
-        <!--  Gazebo Ignition   -->
-        <!-- ================== -->
-        <gazebo reference="world"/>
-        <gazebo>
-            <plugin filename="libign_ros2_control-system.so" name="ign_ros2_control::IgnitionROS2ControlPlugin">
-                <parameters>$(find linear_slider_bringup)/config/linear_slider_controllers.yaml</parameters>
-                <controller_manager_node_name>$(arg prefix)controller_manager</controller_manager_node_name>
-            </plugin>
-        </gazebo>
-    </xacro:if>
 </robot>

File: linear_slider_description/urdf/linear_slider/linear_slider.ros2_control.xacro (robot description, xacro)
@@ -53,6 +53,6 @@
                 </state_interface>
             </joint>
-            <!-- Sensors -->
-            <!-- <sensor name="lim_switch_neg">
+            <!-- Sensors
+            <sensor name="lim_switch_neg">
                 <state_interface name="switch_val">
                     <param name="initial_value">${initial_state['lim_switch_neg']}</param>

File: linear_slider_description/urdf/linear_slider/linear_slider_macro.xacro (robot description, xacro)
@@ -22,4 +22,6 @@
         <xacro:property name="slider_velocity_limit" value="0.25"/>
         <xacro:property name="slider_effort_limit" value="10"/>
+        <!-- tool0 / flange properties -->
+        <xacro:property name="moving_base__flange_offset" value="0.05" />
         <!-- ================== -->
         <!--     Materials      -->
@@ -116,11 +118,16 @@
         <joint name="${prefix}base_joint" type="fixed">
             <parent link="${parent}"/>
-            <child link="${prefix}base_link"/>
+            <child link="${prefix}base"/>
             <xacro:insert_block name="origin"/>
         </joint>
-        <!-- joint1 -->
+        <joint name="${prefix}base_link__base_joint" type="fixed">
+            <origin xyz="0 0 0" rpy="0 0 0"/>
+            <parent link="${prefix}base" />
+            <child link="${prefix}base_link" />
+        </joint>
+        <!-- joint1, moving prismatic joint -->
         <joint name="${prefix}joint1" type="prismatic">
-            <parent link="base_link"/>
-            <child link="moving_base"/>
+            <parent link="${prefix}base_link"/>
+            <child link="${prefix}moving_base"/>
             <axis xyz="1 0 0"/>
             <limit
@@ -130,22 +137,17 @@
                 velocity="${slider_velocity_limit}"
             /> <!-- effort is attribute for enforcing maximum joint effort, between 0 and 100% -->
-            <origin xyz="0.0 0.0 0.0" /> <!-- Define where the joint will be located, defined in terms of parent's reference frame -->
+            <origin xyz="0 0 0" rpy="0 0 0"/> <!-- Define where the joint will be located, defined in terms of parent's reference frame -->
         </joint>
         <!-- Extra joints for ros-industrial standard compatability -->
         <!-- tool frame to fixed frame -->
-        <joint name="${prefix}moving_base-tool0" type="fixed">
+        <joint name="${prefix}moving_base__flange_joint" type="fixed">
             <parent link="${prefix}moving_base"/>
-            <child link="${prefix}tool0"/>
-            <origin xyz="0 0 0" rpy="0 0 0" />
+            <child link="${prefix}flange"/>
+            <origin xyz="0 0 ${moving_base__flange_offset}" rpy="0 0 0" />
         </joint>
-        <joint name="${prefix}base_link-base_joint" type="fixed">
-            <origin xyz="0 0 0" rpy="0 0 0" />
-            <parent link="${prefix}base_link" />
-            <child link="${prefix}base" />
-        </joint>
-        <joint name="${prefix}tool0-flange_joint" type="fixed">
-            <origin xyz="0 0 0" rpy="0 0 0" />
-            <parent link="${prefix}tool0" />
-            <child link="${prefix}flange" />
+        <joint name="${prefix}flange__tool0_joint" type="fixed">
+            <parent link="${prefix}flange" />
+            <child link="${prefix}tool0" />
+            <origin xyz="0 0 0" rpy="0 0 0"/>
         </joint>
     </xacro:macro>

File: linear_slider_moveit/srdf/linear_slider_macro.srdf.xacro (robot description, xacro)
@@ -7,13 +7,18 @@
         <!--CHAINS - When a chain is specified, all the links along the chain (including endpoints) are included in the group. Additionally, all the joints that are parents to included links are also included. This means that joints along the chain and the parent joint of the base link are included in the group-->
         <!--SUBGROUPS - Groups can also be formed by referencing to already defined group names-->
-        <group name="${prefix}${name}_manipulator">
+        <group name="${prefix}manipulator">
+            <!-- <joint name="$(arg prefix)base_joint" />
+            <joint name="$(arg prefix)base_link__base_joint" />
             <joint name="$(arg prefix)joint1"/>
-            <joint name="$(arg prefix)virtual_joint"/>
+            <joint name="$(arg prefix)moving_base__flange_joint" />
+            <joint name="$(arg prefix)flange__tool0_joint" /> -->
             <chain base_link="${prefix}base_link" tip_link="${prefix}flange" />
+            <end_effector name="${prefix}eef" group="${prefix}manipulator" parent_link="${prefix}tool0"/>
         </group>
         <!--GROUP STATES - Purpose - Define a named state for a particular group, in terms of joint values. This is useful to define states like 'folded arms'-->
-        <group_state name="${prefix}center" group="${prefix}${name}_manipulator">
+        <group_state name="${prefix}center" group="${prefix}manipulator">
             <joint name="${prefix}joint1" value="0.0"/>
         </group_state>
+        <virtual_joint name="$(arg prefix)base_joint" type="fixed"  parent_frame="world" child_link="${prefix}base"/>
         <!-- DISABLE COLLISIONS -->
         <disable_collisions link1="${prefix}base_link" link2="${prefix}moving_base" reason="Adjacent"/>
