Commit message: fixed xacro files, added bringup files for joint_state_trajectory

File: linear_slider_description/urdf/linear_slider.urdf.xacro (robot description, xacro)
@@ -4,9 +4,9 @@
     <xacro:arg name="use_mock_hardware" default="false" />
     <xacro:arg name="mock_sensor_commands" default="false" />
-    <xacro:arg name="prefix" default="" />
+    <xacro:arg name="prefix" default="''" />
     <!-- Robot description -->
     <xacro:include filename="$(find linear_slider_description)/urdf/linear_slider/linear_slider_macro.xacro"/>
     <xacro:include filename="$(find linear_slider_description)/urdf/linear_slider/linear_slider.ros2_control.xacro"/>
-    <create />
+    <xacro:linear_slider_macro prefix="$(arg prefix)" />
     <!-- ros2_control -->
     <xacro:linear_slider_ros2_control

File: linear_slider_description/urdf/linear_slider/linear_slider_macro.xacro (robot description, xacro)
@@ -1,5 +1,5 @@
 <?xml version="1.0" encoding="UTF-8"?>
 <robot xmlns:xacro="http://ros.org/wiki/xacro" name="linear_slider">
-    <xacro:macro name="linear_slider" params="prefix">
+    <xacro:macro name="linear_slider_macro" params="prefix">
         <!-- ================== -->
         <!--     Properties     -->

Commit message: got gazebo working!

File: linear_slider_description/urdf/linear_slider.urdf.xacro (robot description, xacro)
@@ -31,5 +31,7 @@
         <!--   Gazebo Classic   -->
         <!-- ================== -->
-        <gazebo reference="world"/>
+        <gazebo reference="$(arg prefix)base_link">
+            <static>true</static>
+        </gazebo>
         <gazebo>
             <plugin filename="libgazebo_ros2_control.so" name="gazebo_ros2_control">

File: linear_slider_description/urdf/linear_slider/linear_slider.ros2_control.xacro (robot description, xacro)
@@ -54,5 +54,5 @@
             </joint>
             <!-- Sensors -->
-            <sensor name="lim_switch_neg">
+            <!-- <sensor name="lim_switch_neg">
                 <state_interface name="switch_val">
                     <param name="initial_value">${initial_state['lim_switch_neg']}</param>
@@ -65,5 +65,5 @@
                 </state_interface>
                 <param name="frame_id">${prefix}base_link</param>
-            </sensor>
+            </sensor> -->
         </ros2_control>
     </xacro:macro>

File: linear_slider_description/urdf/linear_slider/linear_slider_macro.xacro (robot description, xacro)
@@ -11,4 +11,5 @@
         <xacro:property name="frame_height" value="0.25"/>
         <xacro:property name="moving_base_mass" value="10.0" />
+        <xacro:property name="base_link_mass" value="20.0" />
         <!-- Model default position/orientation -->
         <xacro:property name="model_scale" value="0.001 0.001 0.001"/>
@@ -39,5 +40,5 @@
                 <origin rpy="${base_link_start_orientation}" xyz="${start_offset}"/>
                 <geometry>
-                    <mesh filename="package://linear_slider_description/meshes/7thlink_fixed.STL" scale="${model_scale}" />
+                    <mesh filename="file://$(find linear_slider_description)/meshes/7thlink_fixed.STL" scale="${model_scale}" />
                 </geometry>
             </visual>
@@ -52,13 +53,13 @@
             </collision>
             <inertial>
-                <mass value="1000.0" />
+                <mass value="${base_link_mass}" />
                 <origin xyz="0.0 0.0 0.0" />
                 <inertia
-                    ixx="${1*12/(frame_mass + 1000.0) * (frame_width**2 + frame_height**2)}"
+                    ixx="${1*12/(frame_mass + base_link_mass) * (frame_width**2 + frame_height**2)}"
                     ixy="0.0"
                     ixz="0.0"
-                    iyy="${1*12/(frame_mass + 1000.0) * (frame_length**2 + frame_height**2)}"
+                    iyy="${1*12/(frame_mass + base_link_mass) * (frame_length**2 + frame_height**2)}"
                     iyz="0.0"
-                    izz="${1*12/(frame_mass + 1000.0) * (frame_width**2 + frame_length**2)}"
+                    izz="${1*12/(frame_mass + base_link_mass) * (frame_width**2 + frame_length**2)}"
                 />
             </inertial>
@@ -74,5 +75,5 @@
                 <geometry>
                     <mesh
-                        filename="package://linear_slider_description/meshes/7thlink_move.STL"
+                        filename="file://$(find linear_slider_description)/meshes/7thlink_move.STL"
                         scale="${model_scale}"
                     />

Commit message: added parent param to linear_slider

File: linear_slider_description/urdf/linear_slider.urdf.xacro (robot description, xacro)
@@ -1,6 +1,9 @@
 <?xml version="1.0"?>
 <robot xmlns:xacro="https://ros.org/wiki/xacro" name="linear_slider">
+    <!-- World link -->
+    <link name="world" />
     <!-- linear slider -->
     <xacro:include filename="$(find linear_slider_description)/urdf/macro/linear_slider_base.urdf.xacro" />
+    <xacro:arg name="parent" default="world" />
     <xacro:arg name="prefix" default="''" />
     <xacro:arg name="use_mock_hardware" default="false" />
@@ -9,9 +12,10 @@
     <xacro:arg name="sim_gazebo_classic" default="false"/>
     <xacro:linear_slider
-            prefix="$(arg prefix)"
-            sim_gazebo="$(arg sim_gazebo)"
-            sim_gazebo_classic="$(arg sim_gazebo_classic)"
-            use_mock_hardware="$(arg use_mock_hardware)"
-            mock_sensor_commands="$(arg mock_sensor_commands)"
+        parent="$(arg parent)"
+        prefix="$(arg prefix)"
+        sim_gazebo="$(arg sim_gazebo)"
+        sim_gazebo_classic="$(arg sim_gazebo_classic)"
+        use_mock_hardware="$(arg use_mock_hardware)"
+        mock_sensor_commands="$(arg mock_sensor_commands)"
     />
 </robot>

File: linear_slider_description/urdf/macro/linear_slider_base.urdf.xacro (robot description, xacro)
@@ -2,4 +2,5 @@
 <robot xmlns:xacro="http://wiki.ros.org/xacro" name="linear_slider">
     <xacro:macro name="linear_slider" params="
+        parent:='world'
         prefix:=''
         use_mock_hardware:=^|false
@@ -10,12 +11,10 @@
         <!-- Robot description -->
         <xacro:include filename="$(find linear_slider_description)/urdf/macro/linear_slider_macro.xacro"/>
-        <xacro:include filename="$(find linear_slider_description)/urdf/macro/linear_slider.ros2_control.xacro"/>
-        <!-- World link -->
-        <link name="world" />
+        <xacro:include filename="$(find linear_slider_description)/urdf/macro/linear_slider.ros2_control.xacro
         <!-- Macro information -->
         <xacro:linear_slider_macro
             joint_limits_file="$(find linear_slider_description)/config/joint_limits.yaml"
             prefix="${prefix}"
-            parent="world">
+            parent="${parent}">
             <origin xyz="0 0 0" rpy="0 0 0"/>
         </xacro:linear_slider_macro>
