Commit message: updated to moveit configs builder, controller still times out

File: linear_slider_moveit_config/srdf/linear_slider_macro.srdf.xacro (robot description, xacro)
@@ -7,10 +7,6 @@
         <!--CHAINS - When a chain is specified, all the links along the chain (including endpoints) are included in the group. Additionally, all the joints that are parents to included links are also included. This means that joints along the chain and the parent joint of the base link are included in the group-->
         <!--SUBGROUPS - Groups can also be formed by referencing to already defined group names-->
+        <!-- GROUP -->
         <group name="${prefix}manipulator">
-            <!-- <joint name="$(arg prefix)base_joint" />
-            <joint name="$(arg prefix)base_link__base_joint" />
-            <joint name="$(arg prefix)joint1"/>
-            <joint name="$(arg prefix)moving_base__flange_joint" />
-            <joint name="$(arg prefix)flange__tool0_joint" /> -->
             <chain base_link="${prefix}base_link" tip_link="${prefix}flange" />
             <end_effector name="${prefix}eef" group="${prefix}manipulator" parent_link="${prefix}tool0"/>
