Commit message: added dynamic joint limit configuration for URDF, removed additional configuration from moveit package

File: linear_slider_description/urdf/macro/linear_slider_base.urdf.xacro (robot description, xacro)
@@ -14,5 +14,8 @@
         <link name="world" />
         <!-- Macro information -->
-        <xacro:linear_slider_macro prefix="${prefix}" parent="world">
+        <xacro:linear_slider_macro
+            joint_limits_file="$(find linear_slider_description)/config/joint_limits.yaml"
+            prefix="${prefix}"
+            parent="world">
             <origin xyz="0 0 0" rpy="0 0 0"/>
         </xacro:linear_slider_macro>

File: linear_slider_description/urdf/macro/linear_slider_macro.xacro (robot description, xacro)
@@ -1,5 +1,5 @@
 <?xml version="1.0" encoding="UTF-8"?>
 <robot xmlns:xacro="http://ros.org/wiki/xacro" name="linear_slider">
-    <xacro:macro name="linear_slider_macro" params="prefix parent *origin">
+    <xacro:macro name="linear_slider_macro" params="joint_limits_file prefix parent *origin">
         <!-- ================== -->
         <!--     Properties     -->
@@ -24,4 +24,12 @@
         <!-- tool0 / flange properties -->
         <xacro:property name="moving_base__flange_offset" value="0.05" />
+        <!-- Joint limits -->
+        <!-- Yaml file is dynamically built which xacro doesn't handle well, so key is split up and combined as raw string -->
+        <xacro:property name="prefix_part1" value="&#36;"/> <!-- '$' character -->
+        <xacro:property name="prefix_part2" value="(var "/>
+        <xacro:property name="prefix_part3" value="prefix"/>
+        <xacro:property name="prefix_part4" value=")"/>
+        <xacro:property name="joint_name" value="${prefix_part1}${prefix_part2}${prefix_part3}${prefix_part4}joint1"/>
+        <xacro:property name="joint_limits" value="${xacro.load_yaml(joint_limits_file)['joint_limits'][joint_name]}"/>
         <!-- ================== -->
         <!--     Materials      -->
@@ -132,9 +140,9 @@
             <axis xyz="1 0 0"/>
             <limit
-                effort="${slider_effort_limit}"
-                lower="${slider_limit_min}"
-                upper="${slider_limit_max}"
-                velocity="${slider_velocity_limit}"
-            /> <!-- effort is attribute for enforcing maximum joint effort, between 0 and 100% -->
+                lower="${joint_limits['min_position']}"
+                upper="${joint_limits['max_position']}"
+                velocity="${joint_limits['max_velocity']}"
+                effort="${joint_limits['max_acceleration']}" />
+            <!-- effort is attribute for enforcing maximum joint effort, between 0 and 100% -->
             <origin xyz="0 0 0" rpy="0 0 0"/> <!-- Define where the joint will be located, defined in terms of parent's reference frame -->
         </joint>
