Commit message: it turns out the PID values work differently for each hardware setup and mock setup. This is unfortunate.

File: linear_slider_description/urdf/macro/linear_slider.ros2_control.xacro (robot description, xacro)
@@ -20,4 +20,5 @@
                     <plugin>mock_components/GenericSystem</plugin>
                     <param name="mock_sensor_commands">${mock_sensor_commands}</param>
+                    <param name="calculate_dynamics">true</param>
                 </xacro:if>
                 <xacro:if value="${sim_gazebo_classic}">

File: linear_slider_description/urdf/macro/linear_slider_base.urdf.xacro (robot description, xacro)
@@ -2,6 +2,6 @@
 <robot xmlns:xacro="http://wiki.ros.org/xacro" name="linear_slider">
     <xacro:macro name="linear_slider" params="
-        parent:='world'
-        prefix:=''
+        parent:=^|'world'
+        prefix:=^|''
         use_mock_hardware:=^|false
         mock_sensor_commands:=^|false

File: ur_with_linear_slider_bringup/urdf/ur_with_linear_slider.urdf (robot description, URDF)
Before this commit: robot ur_with_linear_slider, 18 links, 17 joints
Joints:
- joint linear_slider__joint1: limit lower=-0.4 upper=0.4 effort=2 velocity=0.25 -> lower=-0.4 upper=0.4 effort=0.2 velocity=0.5
- joint ur_robot__base_joint: parent world -> linear_slider__tool0

File: ur_with_linear_slider_bringup/urdf/ur_with_linear_slider.urdf.xacro (robot description, xacro)
@@ -3,4 +3,6 @@
     <!-- linear slider -->
     <xacro:include filename="$(find linear_slider_description)/urdf/macro/linear_slider_base.urdf.xacro" />
+    <xacro:arg name="linear_slider_parent" default="world"/>
+    <xacro:arg name="linear_slider_robot_ip" default="169.254.57.177"/> <!-- TODO: add this into the macro, but instead get from yaml file-->
     <xacro:arg name="prefix" default="''" />
     <xacro:arg name="use_mock_hardware" default="false" />
@@ -8,10 +10,12 @@
     <xacro:arg name="sim_gazebo" default="false" />
     <xacro:arg name="sim_gazebo_classic" default="false"/>
+    <link name="world"/>
     <xacro:linear_slider
-            prefix="$(arg prefix)"
-            sim_gazebo="$(arg sim_gazebo)"
-            sim_gazebo_classic="$(arg sim_gazebo_classic)"
-            use_mock_hardware="$(arg use_mock_hardware)"
-            mock_sensor_commands="$(arg mock_sensor_commands)"
+        parent="$(arg linear_slider_parent)"
+        prefix="$(arg prefix)"
+        sim_gazebo="$(arg sim_gazebo)"
+        sim_gazebo_classic="$(arg sim_gazebo_classic)"
+        use_mock_hardware="$(arg use_mock_hardware)"
+        mock_sensor_commands="$(arg mock_sensor_commands)"
     />
     <!-- UR robot -->
@@ -33,5 +37,5 @@
     <!-- ros2_control related parameters -->
     <xacro:arg name="headless_mode" default="false" />
-    <xacro:arg name="robot_ip" default="0.0.0.0" />
+    <xacro:arg name="ur_robot_ip" default="0.0.0.0" /> <!-- edited by Luke -->
     <xacro:arg name="script_filename" default=""/>
     <xacro:arg name="output_recipe_filename" default=""/>
@@ -88,5 +92,5 @@
         tool_device_name="$(arg tool_device_name)"
         tool_tcp_port="$(arg tool_tcp_port)"
-        robot_ip="$(arg robot_ip)"
+        robot_ip="$(arg ur_robot_ip)"
         script_filename="$(arg script_filename)"
         output_recipe_filename="$(arg output_recipe_filename)"
