Commit message: ur5+slider trajectory following works. working on servo

File: ur_with_linear_slider_bringup/urdf/ur_with_linear_slider.urdf.xacro (robot description, xacro)
@@ -61,5 +61,5 @@
     <xacro:arg name="simulation_controllers" default="" />
     <!-- initial position for simulations (Fake Hardware, Gazebo, Ignition) -->
-    <xacro:arg name="initial_positions_file" default="$(find ur_description)/config/initial_positions.yaml"/>
+    <xacro:arg name="initial_positions_file" default="$(find ur_with_linear_slider_moveit_config)/config/initial_positions.yaml"/>
     <!-- convert to property to use substitution in function -->
     <xacro:property name="initial_positions_file" default="$(arg initial_positions_file)"/>

File: ur_with_linear_slider_moveit_config/srdf/system.srdf.xacro (robot description, xacro)
@@ -9,4 +9,4 @@
     <xacro:arg name="name" default="ur_with_linear_slider"/>
     <xacro:include filename="$(find ur_with_linear_slider_moveit_config)/srdf/system_macro.srdf.xacro"/>
-    <xacro:ur_with_linear_slider_srdf name="$(arg name)" prefix="$(arg prefix)" tf_prefix="$(arg tf_prefix)"/>
+    <xacro:system_macro name="$(arg name)" prefix="$(arg prefix)" tf_prefix="$(arg tf_prefix)"/>
 </robot>

File: ur_with_linear_slider_moveit_config/srdf/system_macro.srdf.xacro (robot description, xacro)
@@ -1,5 +1,5 @@
 <?xml version="1.0" encoding="UTF-8"?>
 <robot xmlns:xacro="http://wiki.ros.org/xacro">
-    <xacro:macro name="ur_with_linear_slider_srdf" params="name prefix tf_prefix">
+    <xacro:macro name="system_macro" params="name prefix tf_prefix">
         <!--GROUPS - Representation of a set of joints and links. This can be useful for specifying DOF to plan for, defining arms, end effectors, etc-->
         <!--LINKS - When a link is specified, the parent joint of that link (if it exists) is automatically included-->
